File: hardware/combined/combined.kicad_pcb (KiCad board)
At the start: 4 copper layers, 88 x 60 mm, 55 parts, among them J1 Barrel_Jack_MountingPin, J2 Conn_01x03_Pin, J3 Conn_01x02, J4 Conn_Coaxial, J7 Conn_01x02, J8 AudioJack3_SwitchT, J9 AudioJack3_SwitchT, Q1 DMG2305UX, SW1 RotaryEncoder_Switch_MP, U1 LD1117S50TR_SOT223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

Commit message: feat: support for final board design
Connections:
- A1 pad 29: unconnected-(A1-GPIO22-Pad29) -> AMP_~{SHDN}
Routing:
- net AMP_~{SHDN}: track 0.00 -> 54.7 mm
- net GND: vias 275 -> 294
Other:
- board text added: "Designed by nausicaä & kiran"
