File: hardware/combined/combined.kicad_sch (KiCad schematic)
At the start: 55 parts, among them J1 Barrel_Jack_MountingPin, J2 Conn_01x03_Pin, J3 Conn_01x02, J4 Conn_Coaxial, J7 Conn_01x02, J8 AudioJack3_SwitchT, J9 AudioJack3_SwitchT, Q1 DMG2305UX, SW1 RotaryEncoder_Switch_MP, U1 LD1117S50TR_SOT223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

Commit message: feat: support for final board design
Parts:
- C1, C10, C12, C13, C14, C15, C17, C3, C6, C8: MPN (none) -> CL21A106KOQNNNG
- C11, C18, C19, C20, C4, C7, C9: MPN (none) -> 0805ZD104KAT2A
- C2: MPN (none) -> GRM21BR61A226ME51L
- C21, C22, C27: MPN (none) -> 0805X105K160CT
- C23, C24, C25, C26: MPN (none) -> C0603C221J1HACAUTO
- R1: MPN (none) -> RG2012P-104-B-T5
- R2, R3, R4: MPN (none) -> RG2012P-472-D-T5
- R7: MPN (none) -> RG2012P-223-B-T5
- SW1: LCSC C255515 -> C470742; MPN EC11E18244A5 -> EC11E09244BS
Connections:
- net AMP_~{SHDN}: now also A1.29 (GPIO22)
- no-connect marks 13 -> 12
